File: hardware/Comparators.kicad_sch (KiCad schematic)
At the start: 0 parts

Commit message: New BSPD Layout based on BSPD by Jakub Drankiewicz in 2021
-Schematic needs to be adjusted for better understanding
-Comparator of Current Sensor removed, the one on Current Sensor Board is sufficient
Parts:
- added C1, C2, C3: 100n, Capacitor_SMD:C_1206_3216Metric, symbol Device:C
- added D1, D2, D3: D_TVS, Diode_SMD:D_SMB, symbol Device:D_TVS
- added R1, R10, R4, R7: 100k, Resistor_SMD:R_1206_3216Metric, symbol Device:R
- added R11, R12, R13, R3, R6, R8: 10k, Resistor_SMD:R_1206_3216Metric, symbol Device:R
- added RV1, RV2: 20k, Potentiometer_THT:Potentiometer_ACP_CA9-H2,5_Horizontal, symbol Device:R_POT
- added U1, U2: LM393, Package_SO:SOIC-8_3.9x4.9mm_P1.27mm, symbol Comparator:LM393
- added U6: 74AHC1G02, Package_TO_SOT_SMD:SOT-23-5, symbol 74xGxx:74AHC1G02
Connections:
- new net: R7.2, R8.1, U1.2 (-)
- new net: D1.1 (A1), R3.1, U1.3 (+), U1.6 (-)
- new net: RV1.2, U1.5 (+)
- new net: R10.2, R12.1, U2.6 (-)
- new net: D2.1 (A1), R6.1, U2.2 (-), U2.5 (+)
- new net: RV2.2, U2.3 (+)
- new net +5V: C1.1, C2.1, C3.1, R10.1, R11.1, R13.2, R7.1, RV1.1, RV2.1, U1.8 (V+), U2.8 (V+), U6.5 (VCC)
- new net Brake1: R1.1, R3.2
- new net Brake1Logic: R11.2, U1.1, U1.7, U2.1, U2.7, U6.1
- new net Brake2: R4.1, R6.2
- new net CS: D3.1 (A1), R13.1, U6.2
- new net Error: U6.4
- new net GND: C1.2, C2.2, C3.2, D1.2 (A2), D2.2 (A2), D3.2 (A2), R1.2, R12.2, R4.2, R8.2, RV1.3, RV2.3, U1.4 (V-), U2.4 (V-), U6.3 (GND)
Other:
- note added: "1 - nie ok 0 - ok"
- note added: "1 - ok 0 - nie ok"
